File: PCB-KiCAD/DTC/DTC.sch (KiCad schematic (older format))
At the start: 16 parts, among them J1 Conn_01x14, J2 Conn_01x02, J3 Conn_01x02, J4 PJ-102A, J5 Screw_Terminal_01x03, K1 G5LE-1, Q1 BC337, Q2 BC327, U1 NodeMCU1.0(ESP-12E)

Commit message: Updated PCB
Updated PCB and added pdf's of layers
Parts:
- added C1: 100uF, Capacitors_ThroughHole:CP_Radial_D8.0mm_P3.80mm, symbol Device:CP
Connections:
- net at J1.13 (Pin_13), U1.17 (GND): now also J2.1 (Pin_1), J3.2 (Pin_2), J4.2, J4.3, Q1.3 (E), U1.14 (GND), U1.24 (GND), C1.2
- net at K1.1: now also J5.2 (Pin_2); no longer J5.3 (Pin_3)
- net at K1.3: now also J5.3 (Pin_3); no longer J5.2 (Pin_2)
- net at D3.1 (K), K1.5, U1.15 (VIN): now also J4.1, C1.1; no longer J4.3
Changed lines of the file:
@@
 EESchema Schematic File Version 4
+LIBS:DTC-cache
 EELAYER 26 0
 EELAYER END
@@
 	6450 2050 6450 1900
 Wire Wire Line
-	6850 2500 7250 2500
-Wire Wire Line
-	7250 2500 7250 2300
-Wire Wire Line
-	7250 2300 7450 2300
-Wire Wire Line
-	6950 1900 7200 1900
-Wire Wire Line
-	7200 1900 7200 2200
-Wire Wire Line
-	7200 2200 7450 2200
-Wire Wire Line
 	7450 2100 7450 1850
 Wire Wire Line
@@
 Connection ~ 5500 4350
 Wire Wire Line
-	3800 4700 3900 4700
-Wire Wire Line
-	3900 4700 3900 4300
+	3800 4600 3900 4600
 Wire Wire Line
 	3900 4300 3350 4300
@@
 	6700 3950 6700 4100
 Wire Wire Line
-	5250 3150 6100 3150
+	5250 3150 5400 3150
 Wire Wire Line
 	6100 3150 6100 2750
@@
 Wire Wire Line
 	5400 3850 5250 3850
+Wire Wire Line
+	5400 3850 5400 3150
+Connection ~ 5400 3850
+Connection ~ 5400 3150
+Wire Wire Line
+	5400 3150 6100 3150
+Wire Wire Line
+	3650 3850 5250 3850
+Connection ~ 3650 3850
+Connection ~ 5250 3850
+Wire Wire Line
+	7450 2300 7300 2300
+Wire Wire Line
+	7300 2300 7300 1900
+Wire Wire Line
+	7300 1900 6950 1900
+Wire Wire Line
+	6850 2500 7400 2500
+Wire Wire Line
+	7400 2500 7400 2200
+Wire Wire Line
+	7400 2200 7450 2200
+$Comp
+L Device:CP C1
+U 1 1 5CD8E3AB
+P 4350 4600
+F 0 "C1" H 4468 4646 50  0000 L CNN
+F 1 "100uF" H 4468 4555 50  0000 L CNN
+F 2 "Capacitors_ThroughHole:CP_Radial_D8.0mm_P3.80mm" H 4388 4450 50  0001 C CNN
+F 3 "~" H 4350 4600 50  0001 C CNN
+	1    4350 4600
+	1    0    0    -1
+$EndComp
+Wire Wire Line
+	3900 4450 4350 4450
+Connection ~ 3900 4450
+Wire Wire Line
+	3900 4450 3900 4300
+Wire Wire Line
+	4000 4800 4350 4800
+Wire Wire Line
+	4350 4800 4350 4750
+Wire Wire Line
+	3900 4600 3900 4450
+Wire Wire Line
+	3800 4700 3800 4800
+Connection ~ 3800 4800
 $EndSCHEMATC
